File: comprgb.sch (KiCad schematic (older format))
At the start: 42 parts, among them J1 VGA, J2 Conn_01x03_Male, J3 USB_C_Receptacle_Power, J4 SCART_CONN, J5 3xRCA_CONN, U1 MCP1700-2802E_SOT23, U2 LMH1251MT_NOPB, U3 TPF144-VR, U6 74AHC1G86, U7 74AHC1G86

Commit message: bigger gote
Parts:
- added R12, R13: 200, Resistor_SMD:R_0805_2012Metric, symbol Device:R_Small
Connections:
- net labels removed: HSYNC
- wire segments 158 -> 159
Changed lines of the file:
@@
 	4500 1550 4650 1550
-$Comp
-L converted:VCC #PWR0107
-U 1 1 5CC299FA
-P 6100 1850
-F 0 "#PWR0107" H 6100 1700 50  0001 C CNN
-F 1 "VCC" V 6000 1800 50  0000 L CNN
-F 2 "" H 6100 1850 60  0000 C CNN
-F 3 "" H 6100 1850 60  0000 C CNN
-	1    6100 1850
-	0    1    1    0
-$EndComp
-$Comp
-L power:GND #PWR0108
-U 1 1 5CC2A68F
-P 5250 1850
-F 0 "#PWR0108" H 5250 1600 50  0001 C CNN
-F 1 "GND" V 5150 1850 50  0000 R CNN
-F 2 "" H 5250 1850 50  0001 C CNN
-F 3 "" H 5250 1850 50  0001 C CNN
-	1    5250 1850
-	0    1    1    0
-$EndComp
 $Comp
 L ossc:SCART_CONN J4
@@
 Wire Wire Line
 	10200 1600 10200 1800
-Wire Wire Line
-	7350 1700 7650 1700
 Text Label 10550 3400 0    50   ~ 0
 CSYNC
@@
 	0    -1   -1   0
 $EndComp
-Text Label 9050 3300 0    50   ~ 0
-HSYNC
 Wire Wire Line
 	7150 3800 7400 3800
@@
 Wire Wire Line
 	8600 3300 9450 3300
-Text Label 7350 1700 0    50   ~ 0
-HSYNC
 Wire Wire Line
 	2300 5950 2300 6300
@@
 	1    0    0    -1
 $EndComp
+$Comp
+L Device:R_Small R13
+U 1 1 60C75430
+P 7450 1700
+F 0 "R13" V 7650 1650 50  0000 L CNN
+F 1 "200" V 7550 1650 50  0000 L CNN
+F 2 "Resistor_SMD:R_0805_2012Metric" H 7450 1700 50  0001 C CNN
+F 3 "~" H 7450 1700 50  0001 C CNN
+F 4 "C17540" H 7450 1700 50  0001 C CNN "LCSC"
+	1    7450 1700
+	0    -1   -1   0
+$EndComp
+Wire Wire Line
+	7550 1700 7650 1700
+$Comp
+L Device:R_Small R12
+U 1 1 60C780F3
+P 7250 1700
+F 0 "R12" V 7450 1650 50  0000 L CNN
+F 1 "200" V 7350 1650 50  0000 L CNN
+F 2 "Resistor_SMD:R_0805_2012Metric" H 7250 1700 50  0001 C CNN
+F 3 "~" H 7250 1700 50  0001 C CNN
+F 4 "C17540" H 7250 1700 50  0001 C CNN "LCSC"
+	1    7250 1700
+	0    -1   -1   0
+$EndComp
+Wire Wire Line
+	6900 1700 7150 1700
+Text Label 6900 1700 0    50   ~ 0
+CSYNC
+Text Label 9050 3300 0    50   ~ 0
+CSYNC
 $EndSCHEMATC

Commit message: regulator swap, hopefully less shit
Parts:
- J1: symbol ossc:VGA -> comprgb-rescue:VGA-ossc
- J4: symbol ossc:SCART_CONN -> comprgb-rescue:SCART_CONN-ossc
- J5: symbol ossc:3xRCA_CONN -> comprgb-rescue:3xRCA_CONN-ossc
- R2: value 1k33 -> 1k5; LCSC C17382 -> C4310
- U1: value MCP1700-2802E_SOT23 -> AP2125N-1.8TRG1; LCSC C88294 -> C460323
Other:
- note added: "1.8V really LDO -- makes 4.5V"
- note removed: "2.8V really LDO"
Changed lines of the file:
@@
 P 4800 6300
 F 0 "U1" H 4800 6542 50  0000 C CNN
-F 1 "MCP1700-2802E_SOT23" H 4800 6451 50  0000 C CNN
+F 1 "AP2125N-1.8TRG1" H 4800 6451 50  0000 C CNN
 F 2 "Package_TO_SOT_SMD:SOT-23" H 4800 6525 50  0001 C CNN
-F 3 "http://ww1.microchip.com/downloads/en/DeviceDoc/20001826D.pdf" H 4800 6300 50  0001 C CNN
-F 4 "C88294" H 4800 6300 50  0001 C CNN "LCSC"
+F 3 "https://datasheet.lcsc.com/lcsc/1912111437_Diodes-Incorporated-AP2125N-1.8TRG1_C460323.pdf" H 4800 6300 50  0001 C CNN
+F 4 "C460323" H 4800 6300 50  0001 C CNN "LCSC"
 	1    4800 6300
 	1    0    0    -1
@@
 P 5250 6750
 F 0 "R2" H 5309 6796 50  0000 L CNN
-F 1 "1k33" H 5309 6705 50  0000 L CNN
+F 1 "1k5" H 5309 6705 50  0000 L CNN
 F 2 "Resistor_SMD:R_0805_2012Metric" H 5250 6750 50  0001 C CNN
 F 3 "~" H 5250 6750 50  0001 C CNN
-F 4 "C17382" H 5250 6750 50  0001 C CNN "LCSC"
+F 4 "C4310" H 5250 6750 50  0001 C CNN "LCSC"
 	1    5250 6750
 	1    0    0    -1
@@
 $EndComp
 Text Notes 4500 6000 0    50   ~ 0
-2.8V really LDO
+1.8V really LDO -- makes 4.5V
 Wire Wire Line
 	2600 3700 3050 3700
@@
 	4500 1550 4650 1550
 $Comp
-L ossc:SCART_CONN J4
+L comprgb-rescue:SCART_CONN-ossc J4
 U 1 1 5CC3C1EF
 P 8900 1300
@@
 Connection ~ 10200 1400
 $Comp
-L ossc:3xRCA_CONN J5
+L comprgb-rescue:3xRCA_CONN-ossc J5
 U 1 1 5CC742C4
 P 950 3850
@@
 Red
 $Comp
-L ossc:VGA J1
+L comprgb-rescue:VGA-ossc J1
 U 1 1 5CCA16CB
 P 8000 3350

Commit message: add power led, rebuild gerb
Parts:
- added D1: LED, LED_SMD:LED_0805_2012Metric, symbol Device:LED
- added R14: 1k5, Resistor_SMD:R_0805_2012Metric, symbol Device:R_Small
Connections:
- net GND: now also D1.1 (K)
- net VCC: now also R14.2
- new net: D1.2 (A), R14.1
Changed lines of the file:
@@
 Text Label 9050 3300 0    50   ~ 0
 CSYNC
+$Comp
+L Device:R_Small R14
+U 1 1 61A26025
+P 6450 6300
+F 0 "R14" H 6509 6346 50  0000 L CNN
+F 1 "1k5" H 6509 6255 50  0000 L CNN
+F 2 "Resistor_SMD:R_0805_2012Metric" H 6450 6300 50  0001 C CNN
+F 3 "~" H 6450 6300 50  0001 C CNN
+F 4 "C4310" H 6450 6300 50  0001 C CNN "LCSC"
+	1    6450 6300
+	0    1    1    0
+$EndComp
+$Comp
+L Device:LED D1
+U 1 1 61A28116
+P 6650 6650
+F 0 "D1" V 6689 6532 50  0000 R CNN
+F 1 "LED" V 6598 6532 50  0000 R CNN
+F 2 "LED_SMD:LED_0805_2012Metric" H 6650 6650 50  0001 C CNN
+F 3 "~" H 6650 6650 50  0001 C CNN
+	1    6650 6650
+	0    -1   -1   0
+$EndComp
+Wire Wire Line
+	6650 6800 6650 6900
+Wire Wire Line
+	6650 6900 6050 6900
+Wire Wire Line
+	6050 6300 6350 6300
+Wire Wire Line
+	6550 6300 6650 6300
+Wire Wire Line
+	6650 6300 6650 6500
 $EndSCHEMATC

Commit message: swap video amp to THS7374 for parts availability
Parts:
- removed U3: TPF144-VR, Package_SO:MSOP-10_3x3mm_P0.5mm, symbol Videobits:TPF144-VR
- added U3: THS7374, Package_SO:TSSOP-14_4.4x5mm_P0.65mm, symbol Videobits:THS7374
- U1: value AP2125N-1.8TRG1 -> RT9166-18GVL(Z00); LCSC C460323 -> C130827
Connections:
- net GND: now also U3.5 (Gnd), U3.6 (DIS)
- net VCC: now also U3.10 (Vcc), U3.9 (BYP)
- net at C4.2: now also U3.2 (In2)
- net at C5.2: now also U3.3 (In3)
- net at C6.2: now also U3.4 (In4)
- net at R11.2: now also U3.12 (Out3)
- net at R10.2: now also U3.13 (Out2)
- net at R9.2: now also U3.11 (Out4)
Changed lines of the file:
@@
 P 4800 6300
 F 0 "U1" H 4800 6542 50  0000 C CNN
-F 1 "AP2125N-1.8TRG1" H 4800 6451 50  0000 C CNN
+F 1 "RT9166-18GVL(Z00)" H 4800 6451 50  0000 C CNN
 F 2 "Package_TO_SOT_SMD:SOT-23" H 4800 6525 50  0001 C CNN
-F 3 "https://datasheet.lcsc.com/lcsc/1912111437_Diodes-Incorporated-AP2125N-1.8TRG1_C460323.pdf" H 4800 6300 50  0001 C CNN
-F 4 "C460323" H 4800 6300 50  0001 C CNN "LCSC"
+F 3 "https://datasheet.lcsc.com/lcsc/1809281511_Richtek-Tech-RT9166-18GVL-Z00_C130827.pdf" H 4800 6300 50  0001 C CNN
+F 4 "C130827" H 4800 6300 50  0001 C CNN "LCSC"
 	1    4800 6300
 	1    0    0    -1
@@
 Wire Wire Line
 	5550 6900 6050 6900
-Text Label 5000 1350 0    50   ~ 0
-SYNC
-Wire Wire Line
-	5000 1350 5250 1350
 Wire Wire Line
 	4500 1550 4650 1550
@@
 	5400 3000 5350 3000
 $Comp
-L Videobits:TPF144-VR U3
-U 1 1 6009F4CA
-P 5650 1700
-F 0 "U3" H 5675 2559 60  0000 C CNN
-F 1 "TPF144-VR" H 5675 2453 60  0000 C CNN
-F 2 "Package_SO:MSOP-10_3x3mm_P0.5mm" H 5675 2347 60  0000 C CNN
-F 3 "" H 5450 1950 60  0000 C CNN
-F 4 "C155447" H 5650 1700 50  0001 C CNN "LCSC"
-	1    5650 1700
-	1    0    0    -1
-$EndComp
-$Comp
 L Mechanical:Fiducial FID1
 U 1 1 600B9B1B
@@
 Wire Wire Line
 	6650 6300 6650 6500
+$Comp
+L Videobits:THS7374 U3
+U 1 1 628660A0
+P 5450 1450
+F 0 "U3" H 5675 1953 60  0000 C CNN
+F 1 "THS7374" H 5675 1847 60  0000 C CNN
+F 2 "Package_SO:TSSOP-14_4.4x5mm_P0.65mm" H 5450 1450 60  0001 C CNN
+F 3 "" H 5450 1450 60  0000 C CNN
+	1    5450 1450
+	1    0    0    -1
+$EndComp
+$Comp
+L power:GND #PWR0102
+U 1 1 62867621
+P 5250 1850
+F 0 "#PWR0102" H 5250 1600 50  0001 C CNN
+F 1 "GND" H 5255 1677 50  0000 C CNN
+F 2 "" H 5250 1850 50  0001 C CNN
+F 3 "" H 5250 1850 50  0001 C CNN
+	1    5250 1850
+	0    1    1    0
+$EndComp
+$Comp
+L power:VCC #PWR0107
+U 1 1 62867F2C
+P 6100 1850
+F 0 "#PWR0107" H 6100 1700 50  0001 C CNN
+F 1 "VCC" H 6117 2023 50  0000 C CNN
+F 2 "" H 6100 1850 50  0001 C CNN
+F 3 "" H 6100 1850 50  0001 C CNN
+	1    6100 1850
+	0    1    1    0
+$EndComp
 $EndSCHEMATC
