File: comprgb.kicad_sch (KiCad schematic)
At the start: 46 parts, among them J1 VGA, J2 Conn_01x03_Male, J3 USB_C_Receptacle_Power, J4 SCART_CONN, J5 3xRCA_CONN, U1 RT9166-18GVL(Z00), U2 LMH1251MT_NOPB, U3 THS7374, U6 74AHC1G86, U7 74AHC1G86

Commit message: corrected r16/17
Parts:
- R16, R17: LCSC C4310 -> C714010
Changed lines of the file:
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@@
 			)
 		)
-		(property "LCSC" "C4310"
+		(property "LCSC" "C714010"
 			(at 45.72 160.02 0)
 			(effects
@@
 			)
 		)
-		(property "LCSC" "C4310"
+		(property "LCSC" "C714010"
 			(at 45.72 157.48 0)
 			(effects

Commit message: fixed gerbers
Parts:
- R16, R17: LCSC C714010 -> C26023
- U6, U7: LCSC C484740 -> C7471
Changed lines of the file:
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@@
 			)
 		)
-		(property "LCSC" "C484740"
+		(property "LCSC" "C7471"
 			(at 130.81 73.66 0)
 			(effects
@@
 			)
 		)
-		(property "LCSC" "C484740"
+		(property "LCSC" "C7471"
 			(at 130.81 85.09 0)
 			(effects
@@
 			)
 		)
-		(property "LCSC" "C714010"
+		(property "LCSC" "C26023"
 			(at 45.72 160.02 0)
 			(effects
@@
 			)
 		)
-		(property "LCSC" "C714010"
+		(property "LCSC" "C26023"
 			(at 45.72 157.48 0)
 			(effects
