File: comprgb.kicad_sch (KiCad schematic)
At the start: 46 parts, among them J1 VGA, J2 Conn_01x03_Male, J3 USB_C_Receptacle_Power, J4 SCART_CONN, J5 3xRCA_CONN, U1 RT9166-18GVL(Z00), U2 LMH1251MT_NOPB, U3 THS7374, U6 74AHC1G86, U7 74AHC1G86

Commit message: JP21 variant
Parts:
- removed J1: VGA, custom_components:VGA_CONN, symbol comprgb-rescue:VGA-ossc
- removed R8: 75, Resistor_SMD:R_0805_2012Metric, symbol Device:R_Small
- added R15: 200, Resistor_SMD:R_0805_2012Metric, symbol Device:R_Small
Connections:
- net Blue: now also J4.20 (SYNC_IN); no longer J4.7 (RGB_B)
- net GND: now also J4.12 (RSV), J4.3 (AUD_OUT_L), J4.7 (RGB_B), J4.8 (VID_STAT); no longer J4.5 (RGB_B_GND), J4.9 (RGB_G_GND)
- net Green: now also J4.19 (SYNC_OUT); no longer J4.11 (RGB_G)
- net VCC: now also J4.11 (RGB_G), R15.1; no longer J4.8 (VID_STAT)
- net at J4.1 (AUD_OUT_R): no longer JR1.1 (In)
- net at J4.10 (IOCTRL): now also R13.2
- net at J4.16 (RGB_STAT): now also R15.2
- net at J4.2 (AUD_IN_R): now also JU1.1 (In)
- net at J4.6 (AUD_IN_L): now also JR1.1 (In)
- no-connect marks 0 -> 3
Other:
- note added: "Blank"
- note added: "CVBS OUT"
- moved on the sheet: JR1, JU1
