File: comprgb.kicad_pcb (KiCad board)
At the start: 2 copper layers, 50 x 70 mm, 46 parts, among them J1 VGA, J2 Conn_01x03_Male, J3 USB_C_Receptacle_Power, J4 SCART_CONN, J5 3xRCA_CONN, U1 RT9166-18GVL(Z00), U2 LMH1251MT_NOPB, U3 THS7374, U6 74AHC1G86, U7 74AHC1G86

Commit message: updated footprints
Parts:
- moved C14 0.20 mm to (51.6, 61.9)

Commit message: gerbers fixed again
Routing:
- net GND: track 18.0 -> 12.1 mm
Changed lines of the file:
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@@
+	)
+	(segment
+		(start 29.4 86.57)
+		(end 40.47 86.57)
+		(width 0.25)
+		(layer "F.Cu")
+		(net 4)
 	)
 	(segment
@@
 	)
 	(segment
+		(start 40.6 86.7)
+		(end 40.6 88.65)
+		(width 0.25)
+		(layer "F.Cu")
+		(net 4)
+	)
+	(segment
+		(start 48 86.025)
+		(end 50.475 86.025)
+		(width 0.25)
+		(layer "F.Cu")
+		(net 4)
+	)
+	(segment
+		(start 43.5 89.5)
+		(end 47 89.5)
+		(width 0.25)
+		(layer "F.Cu")
+		(net 4)
+	)
+	(segment
 		(start 41.45 89.5)
 		(end 42.8 89.5)
@@
 	)
 	(segment
-		(start 48 86.025)
-		(end 50.475 86.025)
-		(width 0.25)
-		(layer "F.Cu")
-		(net 4)
-	)
-	(segment
-		(start 43.5 89.5)
-		(end 47 89.5)
-		(width 0.25)
-		(layer "F.Cu")
-		(net 4)
-	)
-	(segment
 		(start 53.5 83)
 		(end 53.5 71.373002)
@@
 	)
 	(segment
-		(start 40.17 86.57)
-		(end 40.6 87)
-		(width 0.25)
-		(layer "F.Cu")
-		(net 4)
-	)
-	(segment
 		(start 47.5 68.025)
 		(end 48.525 69.05)
@@
 	)
 	(segment
+		(start 40.6 88.65)
+		(end 41.45 89.5)
+		(width 0.25)
+		(layer "F.Cu")
+		(net 4)
+	)
+	(segment
 		(start 45.625 48.8)
 		(end 45.625 49.6)
@@
 	)
 	(segment
-		(start 40.6 88.65)
-		(end 41.45 89.5)
-		(width 0.25)
-		(layer "F.Cu")
-		(net 4)
-	)
-	(segment
-		(start 29.4 86.57)
-		(end 40.17 86.57)
-		(width 0.25)
-		(layer "F.Cu")
-		(net 4)
-	)
-	(segment
 		(start 43.696 45.142)
 		(end 44.346 45.142)
@@
 	)
 	(segment
+		(start 40.47 86.57)
+		(end 40.6 86.7)
+		(width 0.25)
+		(layer "F.Cu")
+		(net 4)
+	)
+	(segment
 		(start 42.276998 67.95)
 		(end 44 67.95)
@@
 		(start 48.6 57.2)
 		(end 48.6 49.4)
-		(width 0.25)
-		(layer "F.Cu")
-		(net 4)
-	)
-	(segment
-		(start 40.6 87)
-		(end 40.6 88.65)
 		(width 0.25)
 		(layer "F.Cu")
@@
 	)
 	(segment
-		(start 42.55 72.25)
-		(end 41.82501 72.97499)
-		(width 0.25)
-		(layer "F.Cu")
-		(net 6)
-	)
-	(segment
-		(start 40.734315 75.3)
-		(end 41.3 75.3)
-		(width 0.25)
-		(layer "F.Cu")
-		(net 6)
-	)
-	(segment
-		(start 41.82501 72.97499)
-		(end 40.46182 72.97499)
-		(width 0.25)
-		(layer "F.Cu")
-		(net 6)
-	)
-	(segment
 		(start 47.875 70.625)
 		(end 46.65001 71.84999)
@@
 	)
 	(segment
-		(start 39.87501 74.440695)
-		(end 40.734315 75.3)
-		(width 0.25)
-		(layer "F.Cu")
-		(net 6)
-	)
-	(segment
 		(start 52.55 62.1)
 		(end 52.55 64.025)
@@
 	)
 	(segment
-		(start 40.46182 72.97499)
-		(end 39.87501 73.5618)
-		(width 0.25)
-		(layer "F.Cu")
-		(net 6)
-	)
-	(segment
 		(start 46.65001 71.84999)
 		(end 42.95001 71.84999)
-		(width 0.25)
-		(layer "F.Cu")
-		(net 6)
-	)
-	(segment
-		(start 39.87501 73.5618)
-		(end 39.87501 74.440695)
 		(width 0.25)
 		(layer "F.Cu")
@@
 	)
 	(segment
+		(start 38.4 55.85)
+		(end 38.05 55.5)
+		(width 0.25)
+		(layer "F.Cu")
+		(net 34)
+	)
+	(segment
+		(start 45.925 69.85)
+		(end 43.21359 69.85)
+		(width 0.25)
+		(layer "F.Cu")
+		(net 34)
+	)
+	(segment
+		(start 40.625 67.26141)
+		(end 40.625 59.425)
+		(width 0.25)
+		(layer "F.Cu")
+		(net 34)
+	)
+	(segment
 		(start 43.21359 69.85)
 		(end 40.625 67.26141)
@@
 	)
 	(segment
-		(start 45.925 69.85)
-		(end 43.21359 69.85)
+		(start 38.4 57.2)
+		(end 38.4 55.85)
 		(width 0.25)
 		(layer "F.Cu")
@@
 	)
 	(segment
-		(start 38.125001 55.575001)
-		(end 38.05 55.5)
-		(width 0.25)
-		(layer "F.Cu")
-		(net 34)
-	)
-	(segment
-		(start 38.125001 56.925001)
-		(end 38.125001 55.575001)
-		(width 0.25)
-		(layer "F.Cu")
-		(net 34)
-	)
-	(segment
 		(start 40.625 59.425)
-		(end 38.125001 56.925001)
-		(width 0.25)
-		(layer "F.Cu")
-		(net 34)
-	)
-	(segment
-		(start 40.625 67.26141)
-		(end 40.625 59.425)
-		(width 0.25)
-		(layer "F.Cu")
+		(end 38.4 57.2)
+		(width 0.25)
+		(layer "F.Cu")

Commit message: prod files update
Parts:
- moved FID2 5.09 mm to (49.2, 95.5)
Other:
- board text added: "YPbPr to RGB 2026-01-09 rev 1.7 wakabavideo.com"
- board text removed: "YPbPr to RGB 2025-09-13 rev 1.6 wakabavideo.com"
Changed lines of the file:
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@@
 	(footprint "videobits:uwuriel"
 		(layer "F.Cu")
-		(at 53.9 97.45)
+		(at 49.2 95.5)
 		(property "Reference" "FID2"
 			(at 0 0 0)
@@
 		)
 	)
-	(gr_text "YPbPr to RGB\n2025-09-13 rev 1.6\nwakabavideo.com"
+	(gr_text "YPbPr to RGB\n2026-01-09 rev 1.7\nwakabavideo.com"
 		(at 59.3 105.9 0)
 		(layer "F.SilkS")
@@
 	)
 	(segment
-		(start 48.525 69.05)
-		(end 48.525 69.85)
-		(width 0.25)
-		(layer "F.Cu")
-		(net 4)
-	)
-	(segment
 		(start 37.95 54.55)
 		(end 39.81 54.55)
@@
 	)
 	(segment
+		(start 48.525 70.61141)
+		(end 46.53641 72.6)
+		(width 0.25)
+		(layer "F.Cu")
+		(net 4)
+	)
+	(segment
 		(start 44.9 83.2)
 		(end 44.9 84.15)
@@
 	)
 	(segment
-		(start 46.83641 72.3)
-		(end 43.56359 72.3)
-		(width 0.25)
-		(layer "F.Cu")
-		(net 4)
-	)
-	(segment
 		(start 49.175 64.15)
 		(end 49.175 62.725)
@@
 	)
 	(segment
+		(start 46.53641 72.6)
+		(end 43.26359 72.6)
+		(width 0.25)
+		(layer "F.Cu")
+		(net 4)
+	)
+	(segment
 		(start 39.81 54.55)
 		(end 40.11 54.25)
@@
 	)
 	(segment
+		(start 48.525 69.05)
+		(end 48.525 70.61141)
+		(width 0.25)
+		(layer "F.Cu")
+		(net 4)
+	)
+	(segment
 		(start 48 86.025)
 		(end 50.475 86.025)
@@
 	)
 	(segment
-		(start 47.5 68.025)
-		(end 48.525 69.05)
-		(width 0.25)
-		(layer "F.Cu")
-		(net 4)
-	)
-	(segment
 		(start 39.825 54.65)
 		(end 39.81 54.65)
@@
 	)
 	(segment
-		(start 41.86359 74)
-		(end 41.025 74)
+		(start 53.075 70.875)
+		(end 53.075 68.025)
 		(width 0.25)
 		(layer "F.Cu")
@@
 	)
 	(segment
-		(start 53.075 70.875)
-		(end 53.075 68.025)
+		(start 43.26359 72.6)
+		(end 41.86359 74)
 		(width 0.25)
 		(layer "F.Cu")
@@
 	)
 	(segment
+		(start 47.5 68.025)
+		(end 48.525 69.05)
+		(width 0.25)
+		(layer "F.Cu")
+		(net 4)
+	)
+	(segment
 		(start 42.8 87.7625)
 		(end 42.8 89.5)
@@
 	)
 	(segment
+		(start 41.86359 74)
+		(end 41.025 74)
+		(width 0.25)
+		(layer "F.Cu")
+		(net 4)
+	)
+	(segment
 		(start 43.696 45.142)
 		(end 44.346 45.142)
@@
 	)
 	(segment
-		(start 43.56359 72.3)
-		(end 41.86359 74)
-		(width 0.25)
-		(layer "F.Cu")
-		(net 4)
-	)
-	(segment
 		(start 54.66181 48.6)
 		(end 58.10681 45.155)
@@
 	)
 	(segment
-		(start 48.525 69.85)
-		(end 48.525 70.61141)
-		(width 0.25)
-		(layer "F.Cu")
-		(net 4)
-	)
-	(segment
 		(start 48.6 57.2)
 		(end 48.6 49.4)
@@
 	)
 	(segment
-		(start 48.525 70.61141)
-		(end 46.83641 72.3)
-		(width 0.25)
-		(layer "F.Cu")
-		(net 4)
-	)
-	(segment
 		(start 40.11 52.885)
 		(end 39.925 52.7)
@@
 	(segment
 		(start 47.875 70.625)
-		(end 46.65001 71.84999)
+		(end 46.4 72.1)
 		(width 0.25)
 		(layer "F.Cu")
@@
 	)
 	(segment
-		(start 42.95001 71.84999)
-		(end 42.55 72.25)
+		(start 46.4 72.1)
+		(end 42.7 72.1)
 		(width 0.25)
 		(layer "F.Cu")
@@
 	)
 	(segment
-		(start 52.55 62.1)
-		(end 52.55 64.025)
+		(start 47.875 69.85)
+		(end 47.875 70.625)
 		(width 0.25)
 		(layer "F.Cu")
@@
 	)
 	(segment
-		(start 49.825 64.15)
-		(end 53.075 64.15)
+		(start 52.55 62.1)
+		(end 52.55 64.025)
 		(width 0.25)
 		(layer "F.Cu")
@@
 	)
 	(segment
-		(start 46.65001 71.84999)
-		(end 42.95001 71.84999)
+		(start 49.825 64.15)
+		(end 53.075 64.15)
 		(width 0.25)
 		(layer "F.Cu")
@@
 	)
 	(segment
-		(start 47.875 69.85)
-		(end 47.875 70.625)
+		(start 42.7 72.1)
+		(end 42.55 72.25)
 		(width 0.25)
 		(layer "F.Cu")
@@
 	)
 	(segment
-		(start 45.623372 73.851628)
-		(end 45 74.475)
-		(width 0.25)
-		(layer "F.Cu")
-		(net 13)
-	)
-	(segment
-		(start 49.825 69.85)
-		(end 49.825 70.65)
+		(start 49.825 70.65)
+		(end 46.875 73.6)
 		(width 0.25)
 		(layer "F.Cu")
@@
 	)
 	(segment
-		(start 47.274978 73.200022)
-		(end 46.274978 73.200022)
+		(start 45.875 73.6)
+		(end 45 74.475)
 		(width 0.25)
 		(layer "F.Cu")
@@
 	)
 	(segment
-		(start 49.825 70.65)
-		(end 47.274978 73.200022)
+		(start 46.875 73.6)
+		(end 45.875 73.6)
 		(width 0.25)
 		(layer "F.Cu")
@@
 	)
 	(segment
-		(start 46.274978 73.200022)
-		(end 45.623372 73.851628)
+		(start 49.825 69.85)
+		(end 49.825 70.65)
 		(width 0.25)
 		(layer "F.Cu")
@@
 	)
 	(segment
-		(start 43.623372 73.851628)
-		(end 43 74.475)
-		(width 0.25)
-		(layer "F.Cu")
-		(net 15)
-	)
-	(segment
-		(start 49.175 70.65)
-		(end 47.074989 72.750011)
+		(start 49.175 69.85)
+		(end 49.175 70.65)
 		(width 0.25)
 		(layer "F.Cu")
@@
 	)
 	(segment
-		(start 49.175 69.85)
-		(end 49.175 70.65)
+		(start 44.375 73.1)
+		(end 43 74.475)
 		(width 0.25)
 		(layer "F.Cu")
@@
 	)
 	(segment
-		(start 44.724989 72.750011)
-		(end 43.623372 73.851628)
+		(start 49.175 70.65)
+		(end 46.725 73.1)
 		(width 0.25)
 		(layer "F.Cu")
@@
 	)
 	(segment
-		(start 47.074989 72.750011)
-		(end 44.724989 72.750011)
+		(start 46.725 73.1)
+		(end 44.375 73.1)
 		(width 0.25)
 		(layer "F.Cu")
@@
 	)
 	(segment
-		(start 46.575 70.65)
-		(end 46.575 69.85)
+		(start 40.17499 59.6114)
+		(end 40.17499 68.17499)
 		(width 0.25)
 		(layer "F.Cu")
@@
 	)
 	(segment
-		(start 40.17499 68.17499)
-		(end 42.725001 70.725001)
+		(start 42.725001 70.725001)
+		(end 44.876001 70.725001)
 		(width 0.25)
 		(layer "F.Cu")
@@
 	)
 	(segment
-		(start 46.499999 70.725001)
-		(end 46.575 70.65)
+		(start 36.1 57.4)
+		(end 36.9 58.2)
 		(width 0.25)
 		(layer "F.Cu")
@@
 	)
 	(segment
-		(start 40.17499 59.6114)
-		(end 40.17499 68.17499)
+		(start 40.17499 68.17499)
+		(end 42.725001 70.725001)
 		(width 0.25)
 		(layer "F.Cu")
@@
 	)
 	(segment
-		(start 35.380002 55.5)
-		(end 36.1 56.219998)
+		(start 46.575 70.6486)
+		(end 46.575 69.85)
 		(width 0.25)
 		(layer "F.Cu")
@@
 	)
 	(segment
-		(start 36.1 57.4)
-		(end 36.9 58.2)
+		(start 44.876001 70.725001)
+		(end 45.2 71.049)
 		(width 0.25)
 		(layer "F.Cu")
@@
 	)
 	(segment
-		(start 43.452181 70.725001)
-		(end 43.625001 70.725001)
+		(start 35.380002 55.5)
+		(end 36.1 56.219998)
 		(width 0.25)
 		(layer "F.Cu")
@@
 	)
 	(segment
-		(start 43.625001 70.725001)
-		(end 46.499999 70.725001)
+		(start 46.1746 71.049)
+		(end 46.575 70.6486)
 		(width 0.25)
 		(layer "F.Cu")
@@
 	)
 	(segment
-		(start 36.9 58.2)
-		(end 38.76359 58.2)
+		(start 32.19 55.5)
+		(end 35.380002 55.5)
 		(width 0.25)
 		(layer "F.Cu")
@@
 	)
 	(segment
-		(start 32.19 55.5)
-		(end 35.380002 55.5)
+		(start 45.2 71.049)
+		(end 46.1746 71.049)
 		(width 0.25)
 		(layer "F.Cu")
@@
 	)
 	(segment
-		(start 36.1 56.219998)
-		(end 36.1 57.4)
+		(start 36.9 58.2)
+		(end 38.76359 58.2)
 		(width 0.25)
 		(layer "F.Cu")
@@
 	)
 	(segment
-		(start 42.725001 70.725001)
-		(end 43.625001 70.725001)
+		(start 36.1 56.219998)
+		(end 36.1 57.4)
 		(width 0.25)
 		(layer "F.Cu")
@@
 	)
 	(segment
-		(start 47.225 70.63641)
-		(end 46.830705 71.030705)
+		(start 41.425 71.5)
+		(end 46.36141 71.5)
 		(width 0.25)
 		(layer "F.Cu")
@@
 	)
 	(segment
-		(start 46.66141 71.2)
-		(end 46.830705 71.030705)
+		(start 41.125 71.2)
+		(end 41.425 71.5)
 		(width 0.25)
 		(layer "F.Cu")
@@
 	)
 	(segment
-		(start 47.225 69.85)
+		(start 46.36141 71.5)
 		(end 47.225 70.63641)
 		(width 0.25)
@@
 	)
 	(segment
-		(start 41.125 71.2)
-		(end 46.66141 71.2)
+		(start 47.225 70.63641)
+		(end 47.225 69.85)
 		(width 0.25)
 		(layer "F.Cu")

Commit message: prod files updated, trace fixed, jlc placeholder
Routing:
- net VCC: track 146.2 -> 140.5 mm
- net Net-(J4-Pad1): track 32.4 -> 30.9 mm
Other:
- board text added: "JLCJLCJLCJLC"
