File: comprgb.kicad_pcb (KiCad board)
At the start: 2 copper layers, 50 x 70 mm, 46 parts, among them J1 VGA, J2 Conn_01x03_Male, J3 USB_C_Receptacle_Power, J4 SCART_CONN, J5 3xRCA_CONN, U1 RT9166-18GVL(Z00), U2 LMH1251MT_NOPB, U3 THS7374, U6 74AHC1G86, U7 74AHC1G86

Commit message: JP21 variant
Parts:
- removed FID2: Fiducial, videobits:uwuriel
- removed J1: VGA, custom_components:VGA_CONN
- added R15: 200, Resistor_SMD:R_0805_2012Metric, F.Cu at (33.8, 51.2)
Connections:
- J4 pad 1: Net-(J4-Pad1) -> unconnected-(J4-AUD_OUT_R-Pad1)
- J4 pad 10: Net-(J4-Pad10) -> Net-(J4-IOCTRL)
- J4 pad 11: /Green -> VCC
- J4 pad 12: Net-(J4-Pad12) -> GND
- J4 pad 16: Net-(J4-Pad16) -> Net-(J4-RGB_STAT)
- J4 pad 19: Net-(J4-Pad19) -> /Green
- J4 pad 2: Net-(J4-Pad2) -> Net-(J4-AUD_IN_R)
- J4 pad 20: Net-(J4-Pad20) -> /Blue
- J4 pad 3: Net-(J4-Pad3) -> GND
- J4 pad 5: GND -> unconnected-(J4-RGB_B_GND-Pad5)
- J4 pad 6: Net-(J4-Pad6) -> Net-(J4-AUD_IN_L)
- J4 pad 7: /Blue -> GND
- J4 pad 8: VCC -> GND
- J4 pad 9: GND -> unconnected-(J4-RGB_G_GND-Pad9)
- JR1 pad 1: Net-(J4-Pad1) -> Net-(J4-AUD_IN_L)
- JU1 pad 1: Net-(J4-Pad3) -> Net-(J4-AUD_IN_R)
- R13 pad 2: Net-(J4-Pad19) -> Net-(J4-IOCTRL)
- U2 pad 22: Net-(U2-Pad22) -> unconnected-(U2-SD/HD_SELECT-Pad22)
- U3 pad 1: Net-(U3-Pad1) -> unconnected-(U3-In1-Pad1)
- U3 pad 14: Net-(U3-Pad14) -> unconnected-(U3-Out1-Pad14)
- U3 pad 7: Net-(U3-Pad7) -> unconnected-(U3-N/C-Pad7)
- U3 pad 8: Net-(U3-Pad8) -> unconnected-(U3-N/C-Pad8)
Routing:
- net Net-(J4-IOCTRL): track 0.00 -> 37.4 mm
- net Net-(J4-Pad3): track 37.2 -> 0.00 mm
- net Net-(J4-AUD_IN_R): track 0.00 -> 34.4 mm
- net Net-(J4-AUD_IN_L): track 0.00 -> 32.2 mm
- net Net-(J4-Pad1): track 30.9 -> 0.00 mm
- net /VSYNC: track 51.4 -> 24.0 mm, vias 4 -> 2
- net Net-(J4-RGB_STAT): track 0.00 -> 25.1 mm, vias 0 -> 2
- net /CSYNC: track 28.0 -> 4.54 mm
- net Net-(J4-Pad16): track 10.7 -> 0.00 mm
- net /Red: track 16.9 -> 7.67 mm
- net VCC: track 140.5 -> 148.1 mm
- net /Green: track 14.6 -> 20.5 mm
- net Net-(J4-Pad19): track 3.64 -> 0.00 mm
- net /Blue: track 27.6 -> 29.0 mm
Other:
- board text added: "JP21"
